File: 1bitsy-badge.sch (KiCad schematic (older format))
At the start: 5 parts, among them J1 TEENSY-LC, J2 OLED_128x64

Commit message: initial changes
Parts:
- removed J1: TEENSY-LC, Wickerlib:TEENSY-LC, symbol TEENSY-LC
- added S?: SWITCH-TACTILE-SPST-NO-0.05A-12V, B3U-1000P, symbol SWITCH-TACTILE-SPST-NO-0.05A-12V
- added U?: 1bitsy-super-complete, symbol 1bitsy-super-complete
Other:
- moved on the sheet: CAP1, CAP2, CAP3, J2
